File: starbie/starbie.kicad_pcb (KiCad board)
At the start: 2 copper layers, 95.9 x 85.1 mm, 7 parts, among them J1 Conn_01x04_Pin, J2 Conn_01x08_Pin, SW1 SW_Push, SW2 SW_Push, U1 XIAO-ESP32-C3-SMD, U2 DHT11

Commit message: Removed the temporary file
Parts:
- added G***: LOGO, LOGO, B.Cu at (146.4, 88.8)
Other:
- board text added: "PANDABIE v1"
